File: KiCad-Design/KiCad-Design.kicad_pcb (KiCad board)
At the start: 2 copper layers, 43.3 x 33 mm, 69 parts, among them J1 USB_B_Micro, Q1 SI2301, Q2 SI2301, Q3 UMH3N, Q4 SI2307CDS-T1-GE3, U1 PMBT3904, U3 CP2104, U4 LTC4054ES5-4.2, U7 AP2112K-3.3

Commit message: PCB: Updating the PCB design
Parts:
- removed D7: 1N5819, Diode_SMD:D_SOD-123
- removed ESP32: ttgo-32-micro-symbols, ttgo-32-micro:TTGO-32-MICRO
- removed Q1, Q2: SI2301, SI2301:Vishay-S-03946-07_2001-K-0
- removed Q4: SI2307CDS-T1-GE3, SI2307:Vishay-S-03946-07_2001-K-IPC_B
- removed R9: 100K, Resistor_SMD:R_0805_2012Metric
- added U8: AP2112K-3.3, Package_TO_SOT_SMD:SOT-23-5, F.Cu at (231.3, 129.9)
- added U9: ttgo-32-micro, ttgo-32-micro:TTGO-32-MICRO, F.Cu at (242.0, 152.0)
- D1, D2: value 0603ESDA2-TR2 -> 1N4148WS; footprint 0603ESDA2-TR2:Eaton-0603ESDA-0-0-0 -> Diode_SMD:D_SOD-323
- D3: footprint 0603ESDA2-TR2:Eaton-0603ESDA-0-0-0 -> Eaton_0603ESDA2-TR2:Eaton-0603ESDA-0-0-0; moved to B.Cu
- D4: value 1N4148WS -> 0603ESDA2-TR2; footprint Diode_SMD:D_SOD-323 -> Eaton_0603ESDA2-TR2:Eaton-0603ESDA-0-0-0
- D5: value 1N4148WS -> 0603ESDA2-TR2; footprint Diode_SMD:D_SOD-323 -> Eaton_0603ESDA2-TR2:Eaton-0603ESDA-0-0-0; moved to F.Cu
- D6: footprint 0603ESDA2-TR2:Eaton-0603ESDA-0-0-0 -> Eaton_0603ESDA2-TR2:Eaton-0603ESDA-0-0-0
- R1: value 100K -> 33K
- R3: moved to B.Cu
- U1: value PMBT3904 -> TPS2115A; footprint PMBT3904:NXP-PMBT3904,215-0 -> TPS2115A:SON-8; moved to B.Cu
- moved R1 28.5 mm to (234.5, 129.8), turned to 90 degrees
- moved D3 25.4 mm to (227.1, 158.1), turned to 270 degrees
- moved D1 24.4 mm to (231.0, 133.9)
- moved D2 24.3 mm to (233.1, 133.8)
- moved D4 22.7 mm to (231.2, 157.9)
- moved D5 20.1 mm to (252.5, 157.0), turned to 90 degrees
- moved R3 14.4 mm to (238.6, 133.4)
- moved U1 12.5 mm to (237.7, 138.6), turned to 180 degrees
- moved R8 11.6 mm to (236.4, 133.4), turned to 90 degrees
- moved C14 5.89 mm to (247.7, 133.3), turned to 270 degrees
- moved SW3 5.61 mm to (243.4, 136.3)
- moved SW1 5.60 mm to (251.9, 136.4)
- moved SW2 5.60 mm to (247.7, 136.4)
- moved J5 5.20 mm to (257.2, 131.6)
- moved C13 1.87 mm to (251.9, 133.2), turned to 270 degrees
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- renumbered BAT to J2, BUS to J3, External to J4, Sensors to J5, OLED to J6, BLE to SW1, FLASH to SW2, RST to SW3, BME280 to U2, HDC1080 to U5, BME680 to U6
Connections:
- D1 pad 1: Net-(C2-Pad2) -> Net-(D1-Pad1)
- D1 pad 2: GND -> +VSW
- D2 pad 1: Net-(C5-Pad2) -> Net-(D1-Pad1)
- D2 pad 2: GND -> MCU_EN
- D3 pad 1: Net-(D3-Pad1) -> Net-(C2-Pad2)
- D4 pad 1: Net-(D4-Pad1) -> Net-(C5-Pad2)
- D4 pad 2: +5V -> GND
- D5 pad 1: Net-(D4-Pad1) -> Net-(D5-Pad1)
- D5 pad 2: MCU_EN -> GND
- J1 pad 4: Net-(J1-Pad4) -> (no net)
- J2 pad 1: Net-(D3-Pad1) -> Net-(D5-Pad1)
- R1 pad 1: Net-(Q1-Pad1) -> Net-(D1-Pad1)
- R1 pad 2: VCC -> GND
- R19 pad 2: +VSW -> +3.3VA
- R3 pad 2: Net-(Q1-Pad1) -> GND
- R7 pad 1: Net-(D3-Pad1) -> Net-(D5-Pad1)
- R8 pad 1: Net-(D4-Pad1) -> MCU_POWER_MODE
- R8 pad 2: Net-(R8-Pad2) -> VCC
- U1 pad 1: Net-(R8-Pad2) -> MCU_POWER_MODE
- U1 pad 2: GND -> +BATT
- U1 pad 3: Net-(R3-Pad1) -> GND
- U2 pad 2: Net-(U2-Pad2) -> (no net)
- U3 pad 1: Net-(U3-Pad1) -> (no net)
- U3 pad 10: Net-(U3-Pad10) -> (no net)
- U3 pad 11: Net-(U3-Pad11) -> (no net)
- U3 pad 12: Net-(U3-Pad12) -> (no net)
- U3 pad 13: Net-(U3-Pad13) -> (no net)
- U3 pad 14: Net-(U3-Pad14) -> (no net)
- U3 pad 15: Net-(U3-Pad15) -> (no net)
- U3 pad 16: Net-(U3-Pad16) -> (no net)
- U3 pad 17: Net-(U3-Pad17) -> (no net)
- U3 pad 18: Net-(U3-Pad18) -> (no net)
- U3 pad 22: Net-(U3-Pad22) -> (no net)
- U3 pad 24: Net-(U3-Pad24) -> (no net)
- U3 pad 7: +VSW -> +5V
- U3 pad 9: Net-(U3-Pad9) -> (no net)
- U5 pad 3: Net-(U5-Pad3) -> (no net)
- U5 pad 4: Net-(U5-Pad4) -> (no net)
- U5 pad 7: Net-(U5-Pad7) -> (no net)
- U7 pad 4: Net-(U7-Pad4) -> (no net)
Routing:
- net GND: track 402.2 -> 268.7 mm, vias 1 -> 0
- net +VSW: track 89.4 -> 18.3 mm, vias 2 -> 0
- net +5V: track 102.4 -> 53.8 mm, vias 1 -> 4
- net +3V3: track 113.6 -> 78.0 mm, vias 2 -> 4
- net MCU_POWER_MODE: track 0.00 -> 29.1 mm, vias 0 -> 1
- net Net-(Q1-Pad1): track 25.2 -> 0.00 mm
- net MCU_BLE_Adv: track 66.0 -> 45.3 mm
- net +BATT: track 71.2 -> 55.3 mm, vias 1 -> 4
- net MCU_EN: track 9.05 -> 24.6 mm
- net SEN_VCC: track 73.2 -> 58.8 mm, vias 0 -> 1
- net VCC: track 35.1 -> 48.7 mm
- net Net-(D3-Pad1): track 11.1 -> 0.00 mm
- net Net-(D5-Pad1): track 0.00 -> 10.0 mm
- net Net-(D1-Pad1): track 0.00 -> 8.14 mm, vias 0 -> 1
- net +3.3VA: track 0.00 -> 8.13 mm
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- removed copper zone on B.Cu, net GND
- removed copper zone on F.Cu, net GND
- removed copper zone on B.Cu, net SEN_GND
- removed copper zone on F.Cu, net SEN_GND
Other:
- outline, holes or cut-outs redrawn
