File: KiCad-Design/KiCad-Design.kicad_pcb (KiCad board)
At the start: 2 copper layers, 43.3 x 33 mm, 65 parts, among them J1 USB_B_Micro, J2 Battery, J3 SENSOR, J4 Ext, J5 SENSORS, J6 OLED, Q3 UMH3N, SW1 MCU BLE Adv, SW2 MCU FLASH, SW3 MCU RESET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

Commit message: PCB: Updating PCB layout
Parts:
- removed J3: SENSOR, Connector_PinHeader_1.27mm:PinHeader_1x04_P1.27mm_Vertical
- removed J5: SENSORS, Connector_JST:JST_SH_BM04B-SRSS-TB_1x04-1MP_P1.00mm_Vertical
- removed J6: OLED, Connector_PinHeader_2.54mm:PinHeader_1x04_P2.54mm_Vertical
- removed SW1: MCU BLE Adv, Button_Switch_SMD:SW_SPST_CK_RS282G05A3
- added BLE: MCU BLE Adv, Button_Switch_SMD:SW_SPST_CK_RS282G05A3, F.Cu at (251.9, 136.4)
- added BUS: SENSOR, Connector_PinHeader_1.27mm:PinHeader_1x04_P1.27mm_Vertical, F.Cu at (262.5, 147.5)
- added OLED: OLED, Connector_PinHeader_2.54mm:PinHeader_1x04_P2.54mm_Vertical, F.Cu at (238.4, 129.2)
- added SENSOR: SENSORS, Connector_JST:JST_SH_BM04B-SRSS-TB_1x04-1MP_P1.00mm_Vertical, F.Cu at (257.2, 131.6)
- renumbered J2 to BAT, J4 to EXT, SW2 to FLASH, SW3 to RESET
Routing:
- added copper zone on B.Cu, net GND
- added copper zone on F.Cu, net GND
- added copper zone on B.Cu, net SEN_GND
- added copper zone on F.Cu, net SEN_GND
Other:
- outline, holes or cut-outs redrawn
